File: 12V_pwm_pump_and_fan_adaptor_board.kicad_sch (KiCad schematic)
At the start: 0 parts

Commit message: chore: update KiCad project settings and sync internal revision history
Other:
- sheet output_connectors ports: added shared_pwm_signal; removed none
- sheet pwm_input ports: added PWM_input; removed none
Changed lines of the file:
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@@
 	(generator_version "10.0")
 	(paper "A4")
+	(wire
+		(pts
+			(xy 17.78 129.54) (xy 21.59 133.35)
+		)
+		(stroke
+			(width 0)
+			(type default)
+		)
+	)
+	(wire
+		(pts
+			(xy 17.78 101.6) (xy 17.78 129.54)
+		)
+		(stroke
+			(width 0)
+			(type default)
+		)
+	)
+	(wire
+		(pts
+			(xy 27.94 91.44) (xy 17.78 101.6)
+		)
+		(stroke
+			(width 0)
+			(type default)
+		)
+	)
+	(wire
+		(pts
+			(xy 21.59 133.35) (xy 33.02 133.35)
+		)
+		(stroke
+			(width 0)
+			(type default)
+		)
+	)
+	(wire
+		(pts
+			(xy 33.02 91.44) (xy 27.94 91.44)
+		)
+		(stroke
+			(width 0)
+			(type default)
+		)
+	)
 	(sheet
-		(at 27.94 127)
+		(at 33.02 125.73)
 		(size 104.14 33.02)
 		(exclude_from_sim no)
@@
 		)
 		(property "Sheetname" "output_connectors"
-			(at 27.94 126.2884 0)
+			(at 33.02 125.0184 0)
 			(show_name no)
 			(do_not_autoplace no)
@@
 		)
 		(property "Sheetfile" "output_connectors.kicad_sch"
-			(at 27.94 160.6046 0)
+			(at 33.02 159.3346 0)
 			(show_name no)
 			(do_not_autoplace no)
@@
 				)
 				(justify left top)
+			)
+		)
+		(pin "shared_pwm_signal" input
+			(at 33.02 133.35 180)
+			(effects
+				(font
+					(size 1.27 1.27)
+				)
+				(justify left)
 			)
 		)
@@
 			)
 		)
+		(pin "PWM_input" input
+			(at 33.02 91.44 180)
+			(effects
+				(font
+					(size 1.27 1.27)
+				)
+				(justify left)
+			)
+		)
