File: 12V_pwm_fan_output_connector.kicad_sch (KiCad schematic)
At the start: 5 parts, among them J2 Fan_4pin

Commit message: chore: update KiCad project settings and sync internal revision history
Parts:
- added C8: C, Capacitor_SMD:C_0603_1608Metric_Pad1.08x0.95mm_HandSolder, symbol Device:C
- added R2: R, Resistor_SMD:R_0603_1608Metric_Pad0.98x0.95mm_HandSolder, symbol Device:R
Connections:
- net GND: now also C8.2
- net shared_pwm_signal: now also R2.1; no longer J2.4 (PWM)
- new net: C8.1, J2.4 (PWM), R2.2
Other:
- moved on the sheet: J2

Commit message: feat: add Mol connectors and update schematic and PCB designs
Parts:
- C3, C4: footprint Capacitor_SMD:C_1206_3216Metric_Pad1.33x1.80mm_HandSolder -> (none)
- C8: footprint Capacitor_SMD:C_0603_1608Metric_Pad1.08x0.95mm_HandSolder -> (none)
- J2: footprint connectors:0470531000 -> connectors:CONN_SD-47053-001_H10p00_MOL
- R2: footprint Resistor_SMD:R_0603_1608Metric_Pad0.98x0.95mm_HandSolder -> (none)
- TP1: footprint TestPoint:TestPoint_2Pads_Pitch2.54mm_Drill0.8mm -> (none)
Changed lines of the file:
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@@
 			)
 		)
-		(property "Footprint" "Capacitor_SMD:C_1206_3216Metric_Pad1.33x1.80mm_HandSolder"
+		(property "Footprint" ""
 			(at 54.61 25.7048 0)
 			(hide yes)
@@
 		)
 		(property "Value" "+12V"
-			(at 24.13 26.6699 90)
-			(show_name no)
-			(do_not_autoplace no)
-			(effects
-				(font
-					(size 1.27 1.27)
-				)
-				(justify left)
+			(at 26.67 24.13 90)
+			(show_name no)
+			(do_not_autoplace no)
+			(effects
+				(font
+					(size 1.27 1.27)
+				)
 			)
 		)
@@
 			)
 		)
-		(property "Footprint" "connectors:0470531000"
+		(property "Footprint" "connectors:CONN_SD-47053-001_H10p00_MOL"
 			(at 114.3 44.45 0)
 			(hide yes)
@@
 		)
 		(property "Value" "GND"
-			(at 21.59 50.8 0)
-			(show_name no)
-			(do_not_autoplace no)
-			(effects
-				(font
-					(size 1.27 1.27)
-				)
+			(at 24.13 46.9899 0)
+			(show_name no)
+			(do_not_autoplace no)
+			(effects
+				(font
+					(size 1.27 1.27)
+				)
+				(justify left)
 			)
 		)
@@
 			)
 		)
-		(property "Footprint" "Capacitor_SMD:C_0603_1608Metric_Pad1.08x0.95mm_HandSolder"
+		(property "Footprint" ""
 			(at 107.6452 48.26 0)
 			(hide yes)
@@
 		)
 		(property "Value" "GND"
-			(at 90.17 48.2599 90)
-			(show_name no)
-			(do_not_autoplace no)
-			(effects
-				(font
-					(size 1.27 1.27)
-				)
-				(justify right)
+			(at 92.71 44.45 90)
+			(show_name no)
+			(do_not_autoplace no)
+			(effects
+				(font
+					(size 1.27 1.27)
+				)
 			)
 		)
@@
 			)
 		)
-		(property "Footprint" "Resistor_SMD:R_0603_1608Metric_Pad0.98x0.95mm_HandSolder"
+		(property "Footprint" ""
 			(at 100.33 41.148 90)
 			(hide yes)
@@
 			)
 		)
-		(property "Footprint" "TestPoint:TestPoint_2Pads_Pitch2.54mm_Drill0.8mm"
+		(property "Footprint" ""
 			(at 21.59 39.37 0)
 			(hide yes)
@@
 			)
 		)
-		(property "Footprint" "Capacitor_SMD:C_1206_3216Metric_Pad1.33x1.80mm_HandSolder"
+		(property "Footprint" ""
 			(at 54.61 20.6248 0)
 			(hide yes)
